Commit message: Added model colour in RViz

File: ROS/rur_detailed_description/urdf/materials.xacro (robot description, xacro)
@@ -1,6 +1,15 @@
 <?xml version="1.0" ?>
 <robot name="rur_detailed" xmlns:xacro="http://www.ros.org/wiki/xacro" >
-<material name="silver">
-  <color rgba="0.700 0.700 0.700 1.000"/>
+<material name="white">
+  <color rgba="01.00 01.00 01.00 1.000"/>
+</material>
+<material name="blue">
+  <color rgba="00.00 00.00 01.00 1.000"/>
+</material>
+<material name="black">
+  <color rgba="00.00 00.00 00.00 1.000"/>
+</material>
+<material name="grey">
+  <color rgba="00.40 00.40 00.40 1.000"/>
 </material>
 </robot>

File: ROS/rur_detailed_description/urdf/rur_detailed.xacro (robot description, xacro)
@@ -17,5 +17,5 @@
       <mesh filename="package://rur_detailed_description/meshes/base_link.stl" scale="0.001 0.001 0.001"/>
     </geometry>
-    <material name="silver"/>
+    <material name="white"/>
   </visual>
   <collision>
@@ -37,5 +37,5 @@
       <mesh filename="package://rur_detailed_description/meshes/right_wheel.stl" scale="0.001 0.001 0.001"/>
     </geometry>
-    <material name="silver"/>
+    <material name="blue"/>
   </visual>
   <collision>
@@ -57,5 +57,5 @@
       <mesh filename="package://rur_detailed_description/meshes/left_wheel.stl" scale="0.001 0.001 0.001"/>
     </geometry>
-    <material name="silver"/>
+    <material name="blue"/>
   </visual>
   <collision>
@@ -77,5 +77,5 @@
       <mesh filename="package://rur_detailed_description/meshes/right_tyre.stl" scale="0.001 0.001 0.001"/>
     </geometry>
-    <material name="silver"/>
+    <material name="white"/>
   </visual>
   <collision>
@@ -97,5 +97,5 @@
       <mesh filename="package://rur_detailed_description/meshes/left_tyre.stl" scale="0.001 0.001 0.001"/>
     </geometry>
-    <material name="silver"/>
+    <material name="white"/>
   </visual>
   <collision>
@@ -117,5 +117,5 @@
       <mesh filename="package://rur_detailed_description/meshes/front_caster.stl" scale="0.001 0.001 0.001"/>
     </geometry>
-    <material name="silver"/>
+    <material name="blue"/>
   </visual>
   <collision>
@@ -137,5 +137,5 @@
       <mesh filename="package://rur_detailed_description/meshes/back_caster.stl" scale="0.001 0.001 0.001"/>
     </geometry>
-    <material name="silver"/>
+    <material name="blue"/>
   </visual>
   <collision>
@@ -157,5 +157,5 @@
       <mesh filename="package://rur_detailed_description/meshes/lid.stl" scale="0.001 0.001 0.001"/>
     </geometry>
-    <material name="silver"/>
+    <material name="white"/>
   </visual>
   <collision>
@@ -177,5 +177,5 @@
       <mesh filename="package://rur_detailed_description/meshes/lidar.stl" scale="0.001 0.001 0.001"/>
     </geometry>
-    <material name="silver"/>
+    <material name="black"/>
   </visual>
   <collision>
@@ -197,5 +197,5 @@
       <mesh filename="package://rur_detailed_description/meshes/electronics_lid.stl" scale="0.001 0.001 0.001"/>
     </geometry>
-    <material name="silver"/>
+    <material name="blue"/>
   </visual>
   <collision>
@@ -217,5 +217,5 @@
       <mesh filename="package://rur_detailed_description/meshes/long_bar.stl" scale="0.001 0.001 0.001"/>
     </geometry>
-    <material name="silver"/>
+    <material name="grey"/>
   </visual>
   <collision>
@@ -237,5 +237,5 @@
       <mesh filename="package://rur_detailed_description/meshes/head.stl" scale="0.001 0.001 0.001"/>
     </geometry>
-    <material name="silver"/>
+    <material name="white"/>
   </visual>
   <collision>
@@ -257,5 +257,5 @@
       <mesh filename="package://rur_detailed_description/meshes/visor.stl" scale="0.001 0.001 0.001"/>
     </geometry>
-    <material name="silver"/>
+    <material name="blue"/>
   </visual>
   <collision>
@@ -277,5 +277,5 @@
       <mesh filename="package://rur_detailed_description/meshes/monitor_cover.stl" scale="0.001 0.001 0.001"/>
     </geometry>
-    <material name="silver"/>
+    <material name="white"/>
   </visual>
   <collision>
@@ -297,5 +297,5 @@
       <mesh filename="package://rur_detailed_description/meshes/right_ear.stl" scale="0.001 0.001 0.001"/>
     </geometry>
-    <material name="silver"/>
+    <material name="blue"/>
   </visual>
   <collision>
@@ -317,5 +317,5 @@
       <mesh filename="package://rur_detailed_description/meshes/left_ear.stl" scale="0.001 0.001 0.001"/>
     </geometry>
-    <material name="silver"/>
+    <material name="blue"/>
   </visual>
   <collision>
@@ -337,5 +337,5 @@
       <mesh filename="package://rur_detailed_description/meshes/monitor.stl" scale="0.001 0.001 0.001"/>
     </geometry>
-    <material name="silver"/>
+    <material name="black"/>
   </visual>
   <collision>
@@ -357,5 +357,5 @@
       <mesh filename="package://rur_detailed_description/meshes/left_antenna.stl" scale="0.001 0.001 0.001"/>
     </geometry>
-    <material name="silver"/>
+    <material name="blue"/>
   </visual>
   <collision>
@@ -377,5 +377,5 @@
       <mesh filename="package://rur_detailed_description/meshes/right_antenna.stl" scale="0.001 0.001 0.001"/>
     </geometry>
-    <material name="silver"/>
+    <material name="blue"/>
   </visual>
   <collision>
@@ -397,5 +397,5 @@
       <mesh filename="package://rur_detailed_description/meshes/camera_link.stl" scale="0.001 0.001 0.001"/>
     </geometry>
-    <material name="silver"/>
+    <material name="white"/>
   </visual>
   <collision>
@@ -417,5 +417,5 @@
       <mesh filename="package://rur_detailed_description/meshes/realsense.stl" scale="0.001 0.001 0.001"/>
     </geometry>
-    <material name="silver"/>
+    <material name="grey"/>
   </visual>
   <collision>
