Commit message: Made navigation work with simulation

File: ROS/rur_detailed_description/urdf/rur_detailed.xacro (robot description, xacro)
@@ -527,5 +527,5 @@
   <child link="right_antenna"/>
 </joint>
-<joint name="camera_joint" type="revolute">
+<!-- <joint name="camera_joint" type="revolute">
   <origin rpy="0 0 0" xyz="0.07175 -0.072 0.33"/>
   <parent link="head"/>
@@ -533,4 +533,9 @@
   <axis xyz="0.0 1.0 -0.0"/>
   <limit effort="100" lower="-3.141593" upper="3.141593" velocity="100"/>
+</joint> -->
+<joint name="camera_joint" type="fixed">
+  <origin rpy="0 0 0" xyz="0.07175 -0.072 0.33"/>
+  <parent link="head"/>
+  <child link="camera_link"/>
 </joint>
 <joint name="Rigid20" type="fixed">
